Commit message: Your message about the changes

File: xarm_description/urdf/gripper/xarm_gripper.urdf.xacro (robot description, xacro)
@@ -50,5 +50,5 @@
       <child link="${prefix}left_outer_knuckle" />
       <axis xyz="1 0 0" />
-      <limit lower="0" upper="0.85" effort="50" velocity="2" />
+      <limit lower="0" upper="0.85" effort="10" velocity="2" />
     </joint>
     <link name="${prefix}left_finger">
@@ -75,5 +75,5 @@
       <child link="${prefix}left_finger" />
       <axis xyz="-1 0 0" />
-      <limit lower="0" upper="0.85" effort="50" velocity="2" />
+      <limit lower="0" upper="0.85" effort="10" velocity="2" />
       <mimic joint="${prefix}drive_joint" multiplier="1" offset="0" />
     </joint>
@@ -101,5 +101,5 @@
       <child link="${prefix}left_inner_knuckle" />
       <axis xyz="1 0 0" />
-      <limit lower="0" upper="0.85" effort="50" velocity="2" />
+      <limit lower="0" upper="0.85" effort="10" velocity="2" />
       <mimic joint="${prefix}drive_joint" multiplier="1" offset="0" />
     </joint>
@@ -127,5 +127,5 @@
       <child link="${prefix}right_outer_knuckle" />
       <axis xyz="-1 0 0" />
-      <limit lower="0" upper="0.85" effort="50" velocity="2" />
+      <limit lower="0" upper="0.85" effort="10" velocity="2" />
       <mimic joint="${prefix}drive_joint" multiplier="1" offset="0" />
     </joint>
@@ -153,5 +153,5 @@
       <child link="${prefix}right_finger" />
       <axis xyz="1 0 0" />
-      <limit lower="0" upper="0.85" effort="50" velocity="2" />
+      <limit lower="0" upper="0.85" effort="10" velocity="2" />
       <mimic joint="${prefix}drive_joint" multiplier="1" offset="0" />
     </joint>
@@ -179,5 +179,5 @@
       <child link="${prefix}right_inner_knuckle" />
       <axis xyz="-1 0 0" />
-      <limit lower="0" upper="0.85" effort="50" velocity="2" />
+      <limit lower="0" upper="0.85" effort="10" velocity="2" />
       <mimic joint="${prefix}drive_joint" multiplier="1" offset="0" />
     </joint>
@@ -189,3 +189,63 @@
     </joint>
   </xacro:macro>
+<gazebo reference="${prefix}left_finger">
+  <mu1>50.0</mu1>
+  <mu2>50.0</mu2>
+  <kp>0</kp>
+  <kd>0</kd>
+  <soft_cfm>0.001</soft_cfm>
+  <soft_erp>0.8</soft_erp>
+  <max_vel>0.05</max_vel>
+  <min_depth>0.001</min_depth>
+</gazebo>
+<gazebo reference="${prefix}right_finger">
+  <mu1>50.0</mu1>
+  <mu2>50.0</mu2>
+  <kp>0</kp>
+  <kd>0</kd>
+  <soft_cfm>0.001</soft_cfm>
+  <soft_erp>0.8</soft_erp>
+  <max_vel>0.05</max_vel>
+  <min_depth>0.001</min_depth>
+</gazebo>
+<gazebo reference="${prefix}left_outer_knuckle">
+  <mu1>50.0</mu1>
+  <mu2>50.0</mu2>
+  <kp>0</kp>
+  <kd>0</kd>
+  <soft_cfm>0.001</soft_cfm>
+  <soft_erp>0.8</soft_erp>
+  <max_vel>0.05</max_vel>
+  <min_depth>0.001</min_depth>
+</gazebo>
+<gazebo reference="${prefix}right_outer_knuckle">
+  <mu1>50.0</mu1>
+  <mu2>50.0</mu2>
+  <kp>0</kp>
+  <kd>0</kd>
+  <soft_cfm>0.001</soft_cfm>
+  <soft_erp>0.8</soft_erp>
+  <max_vel>0.05</max_vel>
+  <min_depth>0.001</min_depth>
+</gazebo>
+<gazebo reference="${prefix}left_inner_knuckle">
+  <mu1>50.0</mu1>
+  <mu2>50.0</mu2>
+  <kp>0</kp>
+  <kd>0</kd>
+  <soft_cfm>0.001</soft_cfm>
+  <soft_erp>0.8</soft_erp>
+  <max_vel>0.05</max_vel>
+  <min_depth>0.001</min_depth>
+</gazebo>
+<gazebo reference="${prefix}right_inner_knuckle">
+  <mu1>50.0</mu1>
+  <mu2>50.0</mu2>
+  <kp>0</kp>
+  <kd>0</kd>
+  <soft_cfm>0.001</soft_cfm>
+  <soft_erp>0.8</soft_erp>
+  <max_vel>0.05</max_vel>
+  <min_depth>0.001</min_depth>
+</gazebo>
 </robot>

File: xarm_description/urdf/xarm6/xarm6.urdf.xacro (robot description, xacro)
@@ -1,4 +1,4 @@
 <?xml version="1.0"?>
-<robot xmlns:xacro="http://ros.org/wiki/xacro">
+<robot xmlns:xacro="http://ros.org/wiki/xacro" name="xarm6">
   <xacro:macro name="xarm6_urdf" params="prefix
     joint1_lower_limit:=${-2.0*pi}  joint1_upper_limit:=${2.0*pi}
@@ -87,4 +87,10 @@
         origin_rpy="0 0 0" />
     </link>
+    <!-- Attach base link to world with zero rotation -->
+    <!--<joint name="world_to_base" type="fixed">
+      <parent link="world"/>
+      <child link="link_base"/>
+      <origin xyz="0 0 0" rpy="0 0 0"/>
+    </joint>-->
     <joint name="${prefix}joint1" type="revolute">
       <parent link="${prefix}link_base"/>
@@ -244,10 +250,10 @@
       <dynamics damping="1.0" friction="1.0"/>
     </joint>
-    <!-- <link name="${prefix}link_eef" />
+    <!--<link name="${prefix}link_eef" />
     <joint name="${prefix}joint_eef" type="fixed">
       <origin xyz="0 0 0" rpy="0 0 0" />
       <parent link="${prefix}link6" />
       <child link="${prefix}link_eef" />
-    </joint> -->
+    </joint>-->
   </xacro:macro>
 </robot>

File: xarm_description/urdf/xarm_device_macro.xacro (robot description, xacro)
@@ -19,5 +19,5 @@
     ros2_control_params:=''
     load_gazebo_plugin:=false
-    add_realsense_d435i:=false
+    add_realsense_d435i:=true
     add_d435i_links:=true
     use_gazebo_camera:=false
